Commit message: ROS 2 Self-driving car with Ackermann steering

File: urdf/body.xacro (robot description, xacro)
@@ -2,5 +2,5 @@
 <robot xmlns:xacro="http://ros.org/wiki/xacro">
   <xacro:macro name="body_macro" params="suffix parent wheel_radius wheel_base vehicle_mass vehicle_mass_height vehicle_width vehicle_length vehicle_height">
-  <xacro:property name="pi" value="3.1415926835897931" />
+  <!-- <xacro:property name="pi" value="3.1415926835897931" /> -->
     <joint name="${suffix}_joint" type="fixed">
       <parent link="${parent}"/>
@@ -19,9 +19,15 @@
        <origin xyz="0 0 0" rpy="0 0 0"/>
         <geometry>
-          <mesh filename="package://self-driving-car/mesh/body.dae" scale="${wheel_base/2.85} 1 1"/>
+          <mesh filename="package://my_self_driving_bot/mesh/body.dae" scale="${wheel_base/2.85} 1 1"/>
         </geometry>
         <gazebo reference="${suffix}_link">
-  		<material value="Gazebo/Black"/>
-	</gazebo>
+      <visual>
+        <material>
+          <ambient>0.8 0.1 0.1 1</ambient> <!-- Màu đỏ -->
+          <diffuse>0.8 0.1 0.1 1</diffuse>
+          <specular>0.5 0.5 0.5 1</specular>
+        </material>
+      </visual>
+    </gazebo>
       </visual>
       <collision>

File: urdf/monocular_camera.xacro (robot description, xacro)
@@ -1,49 +1,47 @@
 <?xml version="1.0"?>
 <robot xmlns:xacro="http://ros.org/wiki/xacro">
-  <xacro:property name="pi" value="3.1415926835897931" />
   <xacro:macro name="monocular_camera_macro" params="suffix parent namespace x y z roll pitch yaw fps width height fov">
-    <xacro:property name="sensor_box" value="0.05" />
-    <xacro:property name="mass" value="0.1" />
-    <joint name="${suffix}_joint" type="fixed">
-      <origin rpy="${roll} ${pitch} ${yaw}" xyz="${x} ${y} ${z}"/>
-      <parent link="${parent}"/>
-      <child  link="${suffix}_link"/>
-    </joint>
+    <!-- 1. Tạo Link Camera (Khung vỏ camera) -->
     <link name="${suffix}_link">
       <visual>
         <geometry>
-          <box size="${sensor_box} ${sensor_box} ${sensor_box}"/>
+          <box size="0.05 0.05 0.05"/>
         </geometry>
-        <origin rpy="0 0 0" xyz="0 0 0"/>
-        <gazebo reference="${suffix}_link">
-  		<material value="Gazebo/Red"/>
-	</gazebo>
+        <material name="red">
+          <color rgba="1 0 0 1"/>
+        </material>
       </visual>
-      <inertial>
-        <origin rpy="0 0 0" xyz="0 0 0"/>
-        <mass value="${mass}"/>
-        <inertia ixx="${(sensor_box*sensor_box+sensor_box*sensor_box)*mass/12.0}" ixy="0.0" ixz="0.0"
-                 iyy="${(sensor_box*sensor_box+sensor_box*sensor_box)*mass/12.0}" iyz="0.0"
-                 izz="${(sensor_box*sensor_box+sensor_box*sensor_box)*mass/12.0}"/>
-      </inertial>
       <collision>
-        <origin rpy="0 0 0" xyz="0 0 0"/>
         <geometry>
-          <box size="${sensor_box} ${sensor_box} ${sensor_box}"/>
+          <box size="0.05 0.05 0.05"/>
         </geometry>
       </collision>
+      <inertial>
+        <mass value="0.1"/>
+        <inertia ixx="0.0001" ixy="0" ixz="0" iyy="0.0001" iyz="0" izz="0.0001"/>
+      </inertial>
     </link>
+    <!-- 2. Tạo Khớp nối (Gắn camera vào xe) -->
+    <joint name="${suffix}_joint" type="fixed">
+      <parent link="${parent}"/>
+      <child link="${suffix}_link"/>
+      <origin xyz="${x} ${y} ${z}" rpy="${roll} ${pitch} ${yaw}"/>
+    </joint>
+    <!-- 3. Tạo Optical Frame (Quan trọng cho OpenCV) -->
+    <!-- Camera trong ROS nhìn theo trục Z, còn xe nhìn trục X. Cần khớp quay này -->
+    <link name="${suffix}_optical_frame"/>
     <joint name="${suffix}_optical_joint" type="fixed">
-      <origin rpy="${-pi/2} 0 ${-pi/2}" xyz="0 0 0"/>
       <parent link="${suffix}_link"/>
-      <child  link="${suffix}_optical_link"/>
+      <child link="${suffix}_optical_frame"/>
+      <origin xyz="0 0 0" rpy="-1.570796 0 -1.570796"/>
     </joint>
-    <link name="${suffix}_optical_link" />
-    <!-- camera -->
+    <!-- 4. Cấu hình Sensor cho Gazebo Harmonic -->
     <gazebo reference="${suffix}_link">
-      <material value="Gazebo/Black"/>
-      <sensor type="camera" name="${suffix}">
+      <sensor name="${suffix}_sensor" type="camera">
+        <pose>0 0 0 0 0 0</pose>
+        <visualize>true</visualize> <!-- Hiện tia camera trong Gazebo để debug -->
         <update_rate>${fps}</update_rate>
-        <camera name="${suffix}">
+        <topic>camera/image_raw</topic> <!-- Topic gốc trong Gazebo -->
+        <camera>
           <horizontal_fov>${fov}</horizontal_fov>
           <image>
@@ -53,30 +51,8 @@
           </image>
           <clip>
-            <near>0.02</near>
-            <far>300</far>
+            <near>0.1</near>
+            <far>100</far>
           </clip>
-          <noise>
-            <type>gaussian</type>
-            <!-- Noise is sampled independently per pixel on each frame.
-                 That pixel's noise value is added to each of its color
-                 channels, which at that point lie in the range [0,1]. -->
-            <mean>0.0</mean>
-            <stddev>0.007</stddev>
-          </noise>
         </camera>
-        <plugin name="camera_controller" filename="libgazebo_ros_camera.so">
-          <alwaysOn>true</alwaysOn>
-          <updateRate>0.0</updateRate>
-          <cameraName>${namespace}</cameraName>
-          <imageTopicName>image_raw</imageTopicName>
-          <cameraInfoTopicName>camera_info</cameraInfoTopicName>
-          <frameName>${suffix}_optical_link</frameName>
-          <hackBaseline>0.0</hackBaseline>
-          <distortionK1>0.0</distortionK1>
-          <distortionK2>0.0</distortionK2>
-          <distortionK3>0.0</distortionK3>
-          <distortionT1>0.0</distortionT1>
-          <distortionT2>0.0</distortionT2>
-        </plugin>
       </sensor>
     </gazebo>

File: urdf/steering.xacro (robot description, xacro)
@@ -2,5 +2,5 @@
 <robot xmlns:xacro="http://ros.org/wiki/xacro">
   <xacro:macro name="steering_macro" params="suffix parent x y yaw length">
-    <xacro:property name="pi" value="3.1415926835897931" />
+    <!-- <xacro:property name="pi" value="3.1415926835897931" /> -->
     <xacro:property name="radius" value="0.1" />
     <xacro:property name="length" value="0.01" />

File: urdf/vehicle.xacro (robot description, xacro)
@@ -1,15 +1,15 @@
 <?xml version="1.0"?>
 <robot name="autoware_gazebo" xmlns:xacro="http://ros.org/wiki/xacro">
-	<xacro:include filename="$(find self-driving-car)/urdf/body.xacro" />
-	<xacro:include filename="$(find self-driving-car)/urdf/wheel.xacro" />
-	<xacro:include filename="$(find self-driving-car)/urdf/steering.xacro" />
-	<xacro:include filename="$(find self-driving-car)/urdf/monocular_camera.xacro"/>
-	<!--xacro:include filename="$(find self-driving-car)/urdf/imu.xacro"/-->
+	<xacro:include filename="$(find my_self_driving_bot)/urdf/body.xacro" />
+	<xacro:include filename="$(find my_self_driving_bot)/urdf/wheel.xacro" />
+	<xacro:include filename="$(find my_self_driving_bot)/urdf/steering.xacro" />
+	<xacro:include filename="$(find my_self_driving_bot)/urdf/monocular_camera.xacro"/>
+	<!--xacro:include filename="$(find my_self_driving_bot)/urdf/imu.xacro"/-->
 	<xacro:arg name="gpu" default="false"/>
-	<xacro:property name="pi" value="3.1415926835897931"/>
+	<!-- <xacro:property name="pi" value="3.1415926835897931"/> -->
 	<link name="base_footprint"/>
   <!-- ================ vehicle ================ -->
   <!-- load parameter -->
-	<xacro:property name="vehicle_info" value="${load_yaml('$(find self-driving-car)/config/vehicle_info.yaml')}"/>
+	<xacro:property name="vehicle_info" value="${load_yaml('$(find my_self_driving_bot)/config/vehicle_info.yaml')}"/>
   <!-- set parameter -->
 	<xacro:property name="wheel_radius" value="${vehicle_info['wheel_radius']}"/>
@@ -42,9 +42,9 @@
   <xacro:wheel_macro suffix="wheel_left_rear" parent="base_link" x="0" y="${wheel_tread/2}" yaw="0" radius="${wheel_radius}" width="${wheel_width}"/>
   <!-- actuator -->
- 	<xacro:include filename="$(find self-driving-car)/urdf/actuator.xacro"/>
+ 	<!-- <xacro:include filename="$(find my_self_driving_bot)/urdf/actuator.xacro"/> -->
   <!-- gazebo -->
- 	<xacro:include filename="$(find self-driving-car)/urdf/vehicle.gazebo"/>
+ 	<xacro:include filename="$(find my_self_driving_bot)/urdf/vehicle.gazebo"/>
   <!-- ================ sensor ================ -->
-	<xacro:property name="calibration" value="${load_yaml('$(find self-driving-car)/config/calibration.yaml')}"/>
+	<xacro:property name="calibration" value="${load_yaml('$(find my_self_driving_bot)/config/calibration.yaml')}"/>
   <xacro:monocular_camera_macro suffix="camera" parent="base_link" namespace=""
                                 x="${calibration['base_link2camera']['x']}"

File: urdf/wheel.xacro (robot description, xacro)
@@ -2,5 +2,5 @@
 <robot xmlns:xacro="http://ros.org/wiki/xacro">
   <xacro:macro name="wheel_macro" params="suffix parent x y yaw radius width">
-    <xacro:property name="pi" value="3.1415926835897931" />
+    <!-- <xacro:property name="pi" value="3.1415926835897931" /> -->
     <xacro:property name="mass" value="40" />
     <joint name="${suffix}_joint" type="continuous">
@@ -16,5 +16,5 @@
       <visual>
         <geometry>
-          <mesh filename="package://self-driving-car/mesh/wheel.dae" scale="${3*radius} ${3*radius} ${3*radius}"/>
+          <mesh filename="package://my_self_driving_bot/mesh/wheel.dae" scale="${3*radius} ${3*radius} ${3*radius}"/>
         </geometry>
         <origin xyz="0 0 0" rpy="0 0 ${yaw}"/>
